File: sensors.kicad_sch (KiCad schematic)
At the start: 2 parts, among them U2 AHT20, U3 BMP280

Commit message: oscillator + header + connectors
Parts:
- removed U2: AHT20, AHT20:PSON100P300X300X110-6N, symbol AHT20:AHT20
- removed U3: BMP280, Package_LGA:Bosch_LGA-8_2x2.5mm_P0.65mm_ClockwisePinNumbering, symbol Sensor_Pressure:BMP280
