File: SuperDoppler2000.kicad_pcb (KiCad board)
At the start: 2 copper layers, 0 parts

Commit message: Add files via upload
starting layout
Parts:
- added C12: 0.1u, Capacitor_SMD:C_0805_2012Metric_Pad1.18x1.45mm_HandSolder, F.Cu at (155.9, 71.7)
- added C13: 0.1u, Capacitor_SMD:C_0805_2012Metric_Pad1.18x1.45mm_HandSolder, F.Cu at (140.6, 95.7)
- added C14: 10n, Capacitor_SMD:C_0805_2012Metric_Pad1.18x1.45mm_HandSolder, F.Cu at (145.7, 101.0)
- added C15: 1u, Capacitor_SMD:C_0805_2012Metric_Pad1.18x1.45mm_HandSolder, F.Cu at (143.3, 101.0)
- added C16: 1u, Capacitor_SMD:C_0805_2012Metric_Pad1.18x1.45mm_HandSolder, F.Cu at (140.1, 99.9)
- added C17: 4.7u, Capacitor_SMD:C_0805_2012Metric_Pad1.18x1.45mm_HandSolder, B.Cu at (147.3, 84.2)
- added C18: 100n, Capacitor_SMD:C_0805_2012Metric_Pad1.18x1.45mm_HandSolder, B.Cu at (151.1, 102.6)
- added C19: 100n, Capacitor_SMD:C_0805_2012Metric_Pad1.18x1.45mm_HandSolder, B.Cu at (157.7, 102.6)
- added C20: 100n, Capacitor_SMD:C_0805_2012Metric_Pad1.18x1.45mm_HandSolder, B.Cu at (159.7, 93.4)
- added C21: 100n, Capacitor_SMD:C_0805_2012Metric_Pad1.18x1.45mm_HandSolder, B.Cu at (150.1, 91.1)
- added C22: 100n, Capacitor_SMD:C_0805_2012Metric_Pad1.18x1.45mm_HandSolder, B.Cu at (148.5, 95.0)
- added C23: 8pF, Capacitor_SMD:C_0805_2012Metric_Pad1.18x1.45mm_HandSolder, F.Cu at (145.0, 91.8)
- added C24: 8pF, Capacitor_SMD:C_0805_2012Metric_Pad1.18x1.45mm_HandSolder, F.Cu at (145.0, 94.0)
- added CBST1: 100nF, Capacitor_THT:C_Disc_D3.0mm_W1.6mm_P2.50mm, F.Cu at (118.0, 80.9)
- added CR1: DALC208SC6, FootprintLibrary:SOT23-6L_STM, F.Cu at (117.8, 116.8)
- added CR2: D1213A-04TS-7, FootprintLibrary:TSOT26_DIO, F.Cu at (183.7, 97.5)
- added CR3: D1213A-04TS-7, FootprintLibrary:TSOT26_DIO, F.Cu at (182.8, 112.6)
- added Ccomp1: 39nF, Capacitor_THT:C_Disc_D3.0mm_W1.6mm_P2.50mm, F.Cu at (110.2, 96.3)
- added Ccomp2: 68nF, Capacitor_THT:C_Disc_D3.0mm_W1.6mm_P2.50mm, F.Cu at (115.2, 91.4)
- added Cen1: 10nF, Capacitor_THT:C_Disc_D3.0mm_W1.6mm_P2.50mm, F.Cu at (130.6, 77.5)
- added Cin1: 10uF, Capacitor_THT:C_Disc_D3.0mm_W1.6mm_P2.50mm, F.Cu at (122.8, 70.8)
- added Cin2: 10uF, Capacitor_THT:C_Disc_D3.0mm_W1.6mm_P2.50mm, F.Cu at (111.9, 76.9)
- added Cinx1: 100nF, Capacitor_THT:C_Disc_D3.0mm_W1.6mm_P2.50mm, F.Cu at (127.2, 70.9)
- added Cinx2: 100nF, Capacitor_THT:C_Disc_D3.0mm_W1.6mm_P2.50mm, F.Cu at (111.9, 81.1)
- added Cout1: 22uF, Capacitor_THT:C_Disc_D3.0mm_W1.6mm_P2.50mm, F.Cu at (133.5, 74.8)
- added Cout2: 47uF, Capacitor_THT:C_Disc_D3.0mm_W1.6mm_P2.50mm, F.Cu at (118.0, 98.7)
- added Cvcc1: 2.2uF, Capacitor_THT:C_Disc_D3.0mm_W1.6mm_P2.50mm, F.Cu at (111.8, 85.9)
- added D1: ESD9B5.0ST5G, Diode_SMD:D_SOD-323, F.Cu at (111.8, 73.8)
- added D2: BAT60A, Diode_SMD:D_SOD-323, F.Cu at (146.1, 69.4)
- added D3: BAT60A, Diode_SMD:D_SOD-323, F.Cu at (122.2, 99.5)
- added D4: BAT60A, Diode_SMD:D_SOD-323, F.Cu at (168.8, 72.3)
- added D5: GSESLC3V3D323S-2B, Diode_SMD:D_SOD-323_HandSoldering, F.Cu at (180.8, 77.3)
- added D6: GSESLC3V3D323S-2B, Diode_SMD:D_SOD-323_HandSoldering, F.Cu at (172.1, 77.3)
- added D7: GSESLC3V3D323S-2B, Diode_SMD:D_SOD-323_HandSoldering, F.Cu at (176.3, 77.3)
- added DLD2: LED_Red, LED_SMD:LED_0805_2012Metric_Pad1.15x1.40mm_HandSolder, F.Cu at (128.9, 96.7)
- added FB1: FerriteBead, Inductor_SMD:L_0805_2012Metric, F.Cu at (140.2, 102.1)
- added G***: LOGO, graphics:Untitled1, F.Cu at (184.7, 133.8)
- added H1: MountingHole_Pad, MountingHole:MountingHole_3.2mm_M3_Pad, F.Cu at (105.1, 64.9)
- added H2: MountingHole_Pad, MountingHole:MountingHole_3.2mm_M3_Pad, F.Cu at (194.9, 65.3)
- added H3: MountingHole_Pad, MountingHole:MountingHole_3.2mm_M3_Pad, F.Cu at (105.5, 134.7)
- added H4: MountingHole_Pad, MountingHole:MountingHole_3.2mm_M3_Pad, F.Cu at (196.0, 135.9)
- added J1: JST PH, Connector_JST:JST_PH_B2B-PH-K_1x02_P2.00mm_Vertical, F.Cu at (112.7, 63.0)
- added J2: IDC 2x05 2.54mm, FootprintLibrary:SHDR10W66P254_2X5_2019X914X986P, F.Cu at (177.0, 64.3)
- added J3: JST PH, Connector_JST:JST_PH_B3B-PH-K_1x03_P2.00mm_Vertical, F.Cu at (111.0, 111.8)
- added J4: JST PH, Connector_JST:JST_PH_B3B-PH-K_1x03_P2.00mm_Vertical, F.Cu at (111.0, 122.6)
- added J5: JST PH, Connector_JST:JST_PH_B3B-PH-K_1x03_P2.00mm_Vertical, F.Cu at (122.5, 129.6)
- added J6: JST SH, Connector_JST:JST_SH_BM04B-SRSS-TB_1x04-1MP_P1.00mm_Vertical, F.Cu at (194.8, 91.3)
- added J7: JST PH, Connector_JST:JST_PH_B4B-PH-K_1x04_P2.00mm_Vertical, F.Cu at (195.0, 99.0)
- added J8: TBD, Connector_PinHeader_2.54mm:PinHeader_1x04_P2.54mm_Vertical, F.Cu at (196.6, 125.4)
- added J9: TBD, Connector_PinHeader_2.54mm:PinHeader_1x04_P2.54mm_Vertical, F.Cu at (166.2, 125.7)
- added L1: 4.7uH, Inductor_SMD:L_0805_2012Metric, F.Cu at (116.5, 76.7)
- added LD1: LED_Red, LED_SMD:LED_0805_2012Metric_Pad1.15x1.40mm_HandSolder, F.Cu at (140.3, 75.6)
- added LD3: LED_Red, LED_SMD:LED_0805_2012Metric_Pad1.15x1.40mm_HandSolder, F.Cu at (160.5, 72.3)
- added LD4: LED_Green, LED_SMD:LED_0805_2012Metric_Pad1.15x1.40mm_HandSolder, F.Cu at (196.5, 78.1)
- added LD5: LED_Yellow, LED_SMD:LED_0805_2012Metric_Pad1.15x1.40mm_HandSolder, F.Cu at (191.2, 78.5)
- added LD6: LED_Blue, LED_SMD:LED_0805_2012Metric_Pad1.15x1.40mm_HandSolder, F.Cu at (186.9, 78.5)
- added R1: 14.7k, Resistor_SMD:R_0805_2012Metric_Pad1.20x1.40mm_HandSolder, F.Cu at (123.1, 76.0)
- added R10: 4.7k, Resistor_SMD:R_0805_2012Metric_Pad1.20x1.40mm_HandSolder, F.Cu at (153.9, 87.8)
- added R11: 4.7k, Resistor_SMD:R_0805_2012Metric_Pad1.20x1.40mm_HandSolder, F.Cu at (151.7, 87.8)
- added R12: 0, Resistor_SMD:R_0805_2012Metric_Pad1.20x1.40mm_HandSolder, F.Cu at (150.5, 106.2)
- added R13: 100, Resistor_SMD:R_0805_2012Metric_Pad1.20x1.40mm_HandSolder, F.Cu at (195.8, 73.5)
- added R14: 65, Resistor_SMD:R_0805_2012Metric_Pad1.20x1.40mm_HandSolder, F.Cu at (191.7, 73.5)
- added R15: 0, Resistor_SMD:R_0805_2012Metric_Pad1.20x1.40mm_HandSolder, F.Cu at (187.6, 73.8)
- added R16: 10k, Resistor_SMD:R_0805_2012Metric_Pad1.20x1.40mm_HandSolder, F.Cu at (117.8, 111.2)
- added R17: 14k, Resistor_SMD:R_0805_2012Metric_Pad1.20x1.40mm_HandSolder, F.Cu at (118.1, 107.4)
- added R18: 10k, Resistor_SMD:R_0805_2012Metric_Pad1.20x1.40mm_HandSolder, F.Cu at (126.3, 116.7)
- added R19: 14k, Resistor_SMD:R_0805_2012Metric_Pad1.20x1.40mm_HandSolder, F.Cu at (122.5, 116.7)
- added R2: 10kOhms, Resistor_SMD:R_0805_2012Metric_Pad1.20x1.40mm_HandSolder, F.Cu at (126.3, 76.0)
- added R20: 10k, Resistor_SMD:R_0805_2012Metric_Pad1.20x1.40mm_HandSolder, F.Cu at (119.0, 122.5)
- added R21: 14k, Resistor_SMD:R_0805_2012Metric_Pad1.20x1.40mm_HandSolder, F.Cu at (123.3, 122.5)
- added R22: 220, Resistor_SMD:R_0805_2012Metric_Pad1.20x1.40mm_HandSolder, F.Cu at (183.7, 92.9)
- added R23: 220, Resistor_SMD:R_0805_2012Metric_Pad1.20x1.40mm_HandSolder, F.Cu at (183.2, 101.2)
- added R24: 220, Resistor_SMD:R_0805_2012Metric_Pad1.20x1.40mm_HandSolder, F.Cu at (183.2, 105.2)
- added R25: 220, Resistor_SMD:R_0805_2012Metric_Pad1.20x1.40mm_HandSolder, F.Cu at (194.4, 112.6)
- added R26: 220, Resistor_SMD:R_0805_2012Metric_Pad1.20x1.40mm_HandSolder, F.Cu at (191.6, 112.3)
- added R27: 220, Resistor_SMD:R_0805_2012Metric_Pad1.20x1.40mm_HandSolder, F.Cu at (176.8, 112.5)
- added R28: 220, Resistor_SMD:R_0805_2012Metric_Pad1.20x1.40mm_HandSolder, F.Cu at (173.4, 112.3)
- added R3: 220, Resistor_SMD:R_0805_2012Metric_Pad1.20x1.40mm_HandSolder, F.Cu at (177.8, 72.5)
- added R4: 220, Resistor_SMD:R_0805_2012Metric_Pad1.20x1.40mm_HandSolder, F.Cu at (174.1, 72.5)
- added R5: 220, Resistor_SMD:R_0805_2012Metric_Pad1.20x1.40mm_HandSolder, F.Cu at (181.3, 72.5)
- added R6: 220, Resistor_SMD:R_0805_2012Metric_Pad1.20x1.40mm_HandSolder, F.Cu at (183.6, 89.3)
- added R7: 100K, Resistor_SMD:R_0805_2012Metric_Pad1.20x1.40mm_HandSolder, F.Cu at (151.8, 71.8)
- added R8: 150, Resistor_SMD:R_0805_2012Metric_Pad1.20x1.40mm_HandSolder, F.Cu at (164.8, 72.3)
- added R9: 100k, Resistor_SMD:R_0805_2012Metric_Pad1.20x1.40mm_HandSolder, B.Cu at (152.1, 84.0)
- added RLD1: 150, Resistor_SMD:R_0805_2012Metric_Pad1.20x1.40mm_HandSolder, F.Cu at (140.4, 69.2)
- added RLD2: 500, Resistor_SMD:R_0805_2012Metric_Pad1.20x1.40mm_HandSolder, F.Cu at (125.0, 96.7)
- added Rcomp1: 26.7kOhms, Resistor_SMD:R_0805_2012Metric_Pad1.20x1.40mm_HandSolder, F.Cu at (110.4, 92.2)
- added Rfbb1: 48.7kOhms, Resistor_SMD:R_0805_2012Metric_Pad1.20x1.40mm_HandSolder, F.Cu at (125.6, 92.3)
- added Rfbt1: 931kOhms, Resistor_SMD:R_0805_2012Metric_Pad1.20x1.40mm_HandSolder, F.Cu at (125.8, 87.9)
- added SW1: SW_Push, Button_Switch_SMD:SW_SPST_PTS647_Sx50, F.Cu at (153.6, 64.9)
- added U4: STM32L152RETx, Package_QFP:LQFP-64_10x10mm_P0.5mm, F.Cu at (153.9, 97.0)
- added VR1: TPSM863253RDXR, FootprintLibrary:VREG_TPSM863253RDXR, F.Cu at (135.7, 69.4)
- added VR2: TPS61288RQQR, FootprintLibrary:RQQ0011A-MFG, F.Cu at (119.8, 87.1)
- added Y1: MAX7375AXR805, Package_TO_SOT_SMD:SOT-323_SC-70, F.Cu at (143.9, 96.3)
- added Y2: ABS25-32.768KHZ-6-T, Crystal:Crystal_SMD_Abracon_ABS25-4Pin_8.0x3.8mm, F.Cu at (137.1, 90.6)
Routing:
- net +3.3VA: track 0.00 -> 1.00 mm
Other:
- board outline added: 100 x 80 mm
- board text added: "ECE49595 Team2"
- board text added: "SuperDoppler2000"
