File: stm32-L152RE.kicad_sch (KiCad schematic)
At the start: 30 parts, among them J1 Conn_01x04_Pin, J2 JST SH, J4 TDB, J5 TDB, J6 IDC 2x05 2.54mm, J7 Conn_01x02_Pin, SW1 SW_Push, U4 STM32L152RET6, U5 SIT1630AI-S4-DCC-32.768E, Y2 MAX7375AXR805

Commit message: updated schematic
Parts:
- removed J7: Conn_01x02_Pin, symbol Connector:Conn_01x02_Pin
- removed U5: SIT1630AI-S4-DCC-32.768E, FootprintLibrary:SOT_SiT1630-S_SIT, symbol SOT_SiT1630-S_SIT:SIT1630AI-S4-DCC-32.768E
- added C23, C24: 8pF, symbol Device:C
- added D1: BAT60A, Diode_SMD:D_SOD-323, symbol Diode:BAT60A
- added D2: LED, LED_SMD:LED_0805_2012Metric, symbol Device:LED
- added D3, D4, D8: ??, symbol Diode:1N4148WT
- added D5, D6, D7: LED, symbol Device:LED
- added J10: TBD, symbol Connector:Conn_01x04_Pin
- added J11: JST PH, Connector_JST:JST_PH_B2B-PH-K_1x02_P2.00mm_Vertical, symbol Connector_Generic:Conn_01x04
- added J9: JST PH, Connector_JST:JST_PH_B3B-PH-K_1x03_P2.00mm_Vertical, symbol Connector_Generic:Conn_01x03
- added R15: 150, symbol Device:R_US
- added R16, R17, R18: 2k, symbol Device:R_US
- added R19: 10k, symbol Device:R_US
- added R20: 14k, symbol Device:R_US
- added R3: 0, symbol Device:R
- added Y1: ABS25 6pF, Crystal:Crystal_SMD_Abracon_ABS25-4Pin_8.0x3.8mm, symbol Device:Crystal
- J1: value Conn_01x04_Pin -> TBD
- J4, J5: value TDB -> JST PH; footprint (none) -> Connector_JST:JST_PH_B3B-PH-K_1x03_P2.00mm_Vertical
- R7: value 10K -> 100K
Connections:
- net +12V: now also J9.1 (Pin_1)
- net +3.3V: now also R12.2, R13.2, J10.1 (Pin_1), J11.2 (Pin_2); no longer C12.2, C13.1, C14.2, C15.2, C16.1, C16.2, C17.2, C18.2, C19.2, C20.2, C21.2, C22.2, FB2.2, J1.2 (Pin_2), J2.1 (Pin_1), J4.3 (Pin_3), J5.3 (Pin_3), J6.4 (Pin_4), R10.1, R14.1, R8.1, SW1.1, U4.12 (VSSA), U4.18 (VSS), U4.31 (VSS), U4.47 (VSS), U4.63 (VSS), Y2.3 (GND)
- net +3.3VA: now also C16.1, FB2.2
- net NRST: now also J6.1 (Pin_1)
- net at J4.2 (Pin_2), R11.2: now also D4.1 (K)
- net at J5.2 (Pin_2), R9.2: now also D3.1 (K)
- net V_IN_PWR: now reaches J6.10 (Pin_10)
- net GND: now reaches J6.3 (Pin_3)
- net GND: now also C12.2, C13.1, C14.2, C15.2, C16.2, C17.2, C18.2, C19.2, C20.2, C21.2, C22.2, J1.2 (Pin_2), J2.1 (Pin_1), J4.3 (Pin_3), J5.3 (Pin_3), J6.4 (Pin_4), R10.1, R14.1, R8.1, SW1.1, U4.18 (VSS), U4.31 (VSS), U4.47 (VSS), U4.63 (VSS), Y2.3 (GND), C23.1, C24.2, D2.1 (K), D3.2 (A), D4.2 (A), D5.1 (K), D6.1 (K), D7.1 (K), J10.2 (Pin_2), J11.1 (Pin_1), R3.1
- net 3.3V_IN: now reaches J6.7 (Pin_7)
- net 3.3V_IN: now also J6.8 (Pin_8)
- net at J6.9 (Pin_9): now also D1.2 (A)
- net ADC_IN6: now reaches U4.21 (PA5)
- net ADC_IN6: now also R8.2, R9.1
- net ADC_IN7: now reaches U4.22 (PA6)
- net ADC_IN7: now also R10.2, R11.1
- net ADC_IN14: now reaches U4.24 (PC4)
- net ADC_IN14: now also R19.2, R20.1
- net I2C2_SCL: now reaches U4.29 (PB10)
- net I2C2_SCL: now also J11.4 (Pin_4)
- net I2C2_SDA: now reaches U4.30 (PB11)
- net I2C2_SDA: now also J11.3 (Pin_3)
- net PB12: now reaches U4.33 (PB12)
- net PB12: now also R18.1
- net PB13: now reaches U4.34 (PB13)
- net PB13: now also R17.1
- net PB14: now reaches U4.35 (PB14)
- net PB14: now also R16.1
- net USART3_TX: now reaches U4.51 (PC10)
- net USART3_TX: now also J10.3 (Pin_3)
- net USART3_RX: now reaches U4.52 (PC11)
- net USART3_RX: now also J10.4 (Pin_4)
- removed net ADC_IN1: R8.2, R9.1, U4.15 (PA1)
- removed net ADC_IN4: R10.2, R11.1, U4.20 (PA4)
- net USART_RX: no longer names the net of U4.17 (PA3)
- net USART_TX: no longer names the net of U4.16 (PA2)
- new net: D8.2 (A), J9.3 (Pin_3), R19.1
- new net: D6.2 (A), R17.2
- new net: D8.1 (K), J9.2 (Pin_2), R20.2
- new net: D7.2 (A), R18.2
- new net: D2.2 (A), R15.1
- new net: D5.2 (A), R16.2
- new net +4.5_or_+5: D1.1 (K), R15.2
- new net GNDA: R3.2, U4.12 (VSSA)
- new net OSC32_IN: C24.1, Y1.2
- new net OSC32_OUT: C23.2, Y1.1
- no-connect marks 46 -> 34
Other:
- note added: "2 V @ 20mA"
- note added: "3.3V IN not connected??"
- note added: "5V to 3.3V"
- note added: "ADD pull up on IC side"
- note added: "Analog Wind Direction Sensor"
- note added: "Analog Windspeed Senssor"
- note added: "Extra i2c"
- note added: "Extra usart"
- note added: "GPIO for debug"
- note added: "R value seems too low"
- note added: "To boost and buck??"
- note added: "connector: 2.54 mm VS 1.27?"
- note added: "dep. on Cstray?"
- note added: "extra ADC"
- note removed: "10K or 100K?"
- note removed: "2.54 mm VS 1.27 mm?"
- note removed: "3.3V"
- note removed: "5V"
- note removed: "Anenometer (analog)"
- note removed: "GND"
- note removed: "RST"
- note removed: "SWIM"
- note removed: "Wind Dir (analog)"
- note removed: "needs diodes??"
- moved on the sheet: C12, C14, C15, C16, C17, C18, C19, C20, C21, C22, FB2, J1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

Commit message: Add files via upload
starting layout
Parts:
- removed D3, D4, D8: ??, symbol Diode:1N4148WT
- removed J1, J10: TBD, symbol Connector:Conn_01x04_Pin
- removed J11: JST PH, Connector_JST:JST_PH_B2B-PH-K_1x02_P2.00mm_Vertical, symbol Connector_Generic:Conn_01x04
- removed J2: JST SH, Connector_JST:JST_SH_BM04B-SRSS-TB_1x04-1MP_P1.00mm_Vertical, symbol Connector_Generic:Conn_01x04
- removed J4, J5, J9: JST PH, Connector_JST:JST_PH_B3B-PH-K_1x03_P2.00mm_Vertical, symbol Connector_Generic:Conn_01x03
- removed R10, R19, R8: 10k, symbol Device:R_US
- removed R11, R20, R9: 14k, symbol Device:R_US
- removed R3: 0, symbol Device:R
- removed Y1: ABS25 6pF, Crystal:Crystal_SMD_Abracon_ABS25-4Pin_8.0x3.8mm, symbol Device:Crystal
- added D5, D6, D7: GSESLC3V3D323S-2B, Diode_SMD:D_SOD-323_HandSoldering, symbol Diode:ESD9B3.3ST5G
- added H1, H2, H3, H4: MountingHole_Pad, MountingHole:MountingHole_3.2mm_M3_Pad, symbol Mechanical:MountingHole_Pad
- added R12: 0, Resistor_SMD:R_0805_2012Metric_Pad1.20x1.40mm_HandSolder, symbol Device:R_US
- added R3, R4, R5: 220, Resistor_SMD:R_0805_2012Metric_Pad1.20x1.40mm_HandSolder, symbol Device:R_US
- added Y2: ABS25-32.768KHZ-6-T, Crystal:Crystal_SMD_Abracon_ABS25-4Pin_8.0x3.8mm, symbol ABS25-32_768KHZ-6-T:ABS25-32.768KHZ-6-T
- C12, C13, C14, C15, C16, C17, C18, C19, C20, C21, C22, C23, C24: footprint (none) -> Capacitor_SMD:C_0805_2012Metric_Pad1.18x1.45mm_HandSolder
- FB1: renamed from FB2; footprint (none) -> Inductor_SMD:L_0805_2012Metric
- J2: renamed from J6; footprint Connector_IDC:IDC-Header_2x05_P2.54mm_Latch_Vertical -> FootprintLibrary:SHDR10W66P254_2X5_2019X914X986P
- LD3: renamed from D2; value LED -> LED_Red; footprint LED_SMD:LED_0805_2012Metric -> LED_SMD:LED_0805_2012Metric_Pad1.15x1.40mm_HandSolder
- LD4: renamed from D7; value LED -> LED_Green; footprint (none) -> LED_SMD:LED_0805_2012Metric_Pad1.15x1.40mm_HandSolder
- LD5: renamed from D5; value LED -> LED_Yellow; footprint (none) -> LED_SMD:LED_0805_2012Metric_Pad1.15x1.40mm_HandSolder
- LD6: renamed from D6; value LED -> LED_Blue; footprint (none) -> LED_SMD:LED_0805_2012Metric_Pad1.15x1.40mm_HandSolder
- R10: renamed from R12; footprint (none) -> Resistor_SMD:R_0805_2012Metric_Pad1.20x1.40mm_HandSolder
- R11: renamed from R13; footprint (none) -> Resistor_SMD:R_0805_2012Metric_Pad1.20x1.40mm_HandSolder
- R13: renamed from R18; value 2k -> 100; footprint (none) -> Resistor_SMD:R_0805_2012Metric_Pad1.20x1.40mm_HandSolder
- R14: renamed from R16; value 2k -> 65; footprint (none) -> Resistor_SMD:R_0805_2012Metric_Pad1.20x1.40mm_HandSolder
- R15: renamed from R17; value 2k -> 0; footprint (none) -> Resistor_SMD:R_0805_2012Metric_Pad1.20x1.40mm_HandSolder
- R7: footprint (none) -> Resistor_SMD:R_0805_2012Metric_Pad1.20x1.40mm_HandSolder
- R8: renamed from R15; footprint (none) -> Resistor_SMD:R_0805_2012Metric_Pad1.20x1.40mm_HandSolder
- R9: renamed from R14; footprint (none) -> Resistor_SMD:R_0805_2012Metric_Pad1.20x1.40mm_HandSolder
- SW1: footprint (none) -> Button_Switch_SMD:SW_SPST_PTS647_Sx50
- U4: value STM32L152RET6 -> STM32L152RETx
- renumbered D1 to D4, Y2 to Y1
Connections:
- net RCC_OSC32_IN is gone; now on net OSC32_IN: U4.3 (PC14)
- net RCC_OSC32_OUT is gone; now on net OSC32_OUT: U4.4 (PC15)
- net V_IN_PWR is gone; now on an unnamed net: J2.10 (Pin_10)
- net GND: now also D5.1 (A1), D6.1 (A1), D7.1 (A1), R12.1
- net GNDA: now also R12.2
- net NRST: now also D5.2 (A2), R5.1; no longer J2.1 (Pin_1)
- net OSC32_IN: now also C23.2, Y2.1 (CRYSTAL_1), Y2.2 (NC_1); no longer C24.1
- net OSC32_OUT: now also C24.1, Y2.3 (NC_2), Y2.4 (CRYSTAL_2); no longer C23.2
- net SWCLK: now also D7.2 (A2), R4.2; no longer J2.6 (Pin_6)
- net SWDIO: now also D6.2 (A2), R3.2; no longer J2.2 (Pin_2)
- net at D4.2 (A): no longer J2.9 (Pin_9)
- net 3.3V_IN: no longer names the net of J2.7 (Pin_7)
- net 3.3V_IN: no longer J2.8 (Pin_8)
- net I2C1_SCL renamed I2C1SCL
- new net: J2.1 (Pin_1), R5.2
- new net: J2.6 (Pin_6), R4.1
- new net: J2.2 (Pin_2), R3.1
- no-connect marks 34 -> 36
Other:
- added sheet Peripherals (peripherals.kicad_sch)
- note added: "2.1V @ 10mA"
- note added: "3.1V @ 10mA"
- note added: "placehodler footprint"
- note removed: "3.3V IN not connected??"
- note removed: "5V to 3.3V"
- note removed: "ADD pull up on IC side"
- note removed: "Analog Wind Direction Sensor"
- note removed: "Analog Windspeed Senssor"
- note removed: "BME280"
- note removed: "HM10 Bluetooth Module"
- note removed: "need to add: extra GPIO status LEDS debug connection points"
- moved on the sheet: C23, C24, D4, J2, LD3, LD4, LD5, LD6, R11, R13, R14, R15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
